Commit message: drive bot rviz

File: description/robot_core.xacro (robot description, xacro)
@@ -2,4 +2,5 @@
 <robot xmlns:xacro="http://www.ros.org/wiki/xacro"  name="robot">
     <xacro:include filename="inertial_macros.xacro"/>
+    <xacro:include filename="gazebo_control.xacro"/>
     <!-- Example materials -->
     <!-- here material, color are called tags -->
@@ -50,4 +51,7 @@
         </xacro:inertial_box>
     </link>
+    <gazebo reference="chassis">
+        <material>Gazebo/White</material>
+    </gazebo>
     <!-- Left Wheel -->
     <joint name = "left_wheel_joint" type="continuous">
@@ -75,4 +79,7 @@
         </xacro:inertial_cylinder>
     </link>
+    <gazebo reference="left_wheel">
+        <material>Gazebo/Black</material>
+    </gazebo>
     <!-- Right Wheel -->
     <joint name = "right_wheel_joint" type="continuous">
@@ -100,4 +107,7 @@
         </xacro:inertial_cylinder>
     </link>
+    <gazebo reference="right_wheel">
+        <material>Gazebo/Black</material>
+    </gazebo>
     <joint name="caster_wheel_joint" type="fixed">
         <parent link="chassis"/>
@@ -121,3 +131,8 @@
         </xacro:inertial_sphere>
     </link>
+    <gazebo reference="caster_wheel">
+        <material>Gazebo/Red</material>
+        <mu1 value = "0.001"/>
+        <mu2 value = "0.001"/>
+    </gazebo>
 </robot>
